File: bluejack.kicad_pcb (KiCad board)
At the start: 4 copper layers, 37.3 x 46.8 mm, 6 parts, among them J1 AudioPlug2, J2 BLE HC-08, J3 USB_B_Micro, U1 ATtiny814-SS

Commit message: First ideas
Parts:
- moved J2 9.04 mm to (137.5, 52.0), turned to 0 degrees
Routing:
- net DIG: track 0.00 -> 16.5 mm
- net BLE_RX: track 19.7 -> 30.8 mm
- net +3V3: track 3.32 -> 10.0 mm
- net BLE_TX: track 18.2 -> 24.1 mm
- net GND: track 28.3 -> 31.8 mm
