File: bluejack.kicad_sch (KiCad schematic)
At the start: 7 parts, among them J1 AudioPlug2, J2 BLE HC-08, J3 USB_B_Micro, J4 AudioPlug3, U1 ATtiny814-SS

Commit message: First ideas
Other:
- moved on the sheet: J4
Changed lines of the file:
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@@
 	(symbol
 		(lib_id "Connector_Audio:AudioPlug3")
-		(at 105.41 31.75 0)
+		(at 106.68 31.75 0)
 		(unit 1)
 		(exclude_from_sim no)
@@
 		(fields_autoplaced yes)
 		(property "Reference" "J4"
-			(at 105.41 21.59 0)
+			(at 106.68 21.59 0)
 			(effects
 				(font
@@
 		)
 		(property "Value" "AudioPlug3"
-			(at 105.41 24.13 0)
+			(at 106.68 24.13 0)
 			(effects
 				(font
@@
 		)
 		(property "Footprint" ""
-			(at 107.95 33.02 0)
+			(at 109.22 33.02 0)
 			(effects
 				(font
@@
 		)
 		(property "Datasheet" "~"
-			(at 107.95 33.02 0)
+			(at 109.22 33.02 0)
 			(effects
 				(font
@@
 		)
 		(property "Description" "Audio Jack, 3 Poles (Stereo / TRS)"
-			(at 105.41 31.75 0)
+			(at 106.68 31.75 0)
 			(effects
 				(font
